Commit message: fixed camera and other stuff

File: rosbot_ros/rosbot_description/urdf/rosbot.xacro (robot description, xacro)
@@ -236,13 +236,13 @@
   </transmission>
   <!-- Orbbec Astra RGBD Camera -->
-  <joint name="astra_joint" type="continuous">
-    <axis xyz="0 0 1" />
+  <joint name="astra_joint" type="fixed">
+    <axis xyz="0 0 0" />
     <origin xyz="-0.03 0 0.18" rpy="0 0 0"/>
     <parent link="body_link"/>
     <child link="camera_link"/>
-    <limit effort="1" velocity="10"/>
-    <joint_properties damping="5.0" friction="1.0"/>
-  </joint>
-  <transmission name="astra_joint_trans">
+    <!-- <limit effort="1" velocity="10"/>
+    <joint_properties damping="5.0" friction="1.0"/> -->
+  </joint>
+  <!-- <transmission name="astra_joint_trans">
     <type>transmission_interface/SimpleTransmission</type>
     <joint name="astra_joint">
@@ -253,5 +253,5 @@
       <mechanicalReduction>1</mechanicalReduction>
     </actuator>
-  </transmission>
+  </transmission> -->
   <link name="camera_link">
     <collision>
